File: hardware/board-study/frother-board.kicad_sch (KiCad schematic)
At the start: 23 parts, among them K1 Power button, M1 Motor, U1 unmarked

Commit message: U1 pin readings: pin 2 = BAT, pin 8 = GND; 3.6 ohm short between them
- power-section: U1.2 BAT+ and U1.8 GND measured and verified;
  C1.1 now inferred BAT+; schematic regenerated (draft-3)
- u1-candidates: measured pin table; CX3320, CX3358B, CX3318B ruled
  out; WD8001 still consistent
- repair log follows in #5 comment

Refs #5, #9, #12

Co-Authored-By: Claude Opus 5.5 (1M context) <noreply@anthropic.com>
Connections:
- net U1_PIN2? is gone; now on net BAT+: C1.1, U1.2
- net GND: now also U1.8
Changed lines of the file:
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@@
     (title "Frother Board KD-F316-V1.0 - Board study")
     (date "2026-10-11")
-    (rev "draft-2")
+    (rev "draft-3")
     (comment 1 "Power (#9), Motor drive (#10), Button and LEDs (#11). Traced from photos; unverified.")
   )
@@
     (pin "1") (pin "2"))
   (wire (pts (xy 147.32 72.39) (xy 147.32 67.31)) (stroke (width 0) (type default) (color 0 0 0 0)))
-  (label "U1_PIN2?" (at 147.32 67.31 90) (effects (font (size 1.27 1.27)) (justify left bottom)))
+  (label "BAT+" (at 147.32 67.31 90) (effects (font (size 1.27 1.27)) (justify left bottom)))
   (wire (pts (xy 147.32 80.01) (xy 147.32 85.09)) (stroke (width 0) (type default) (color 0 0 0 0)))
   (label "GND" (at 147.32 85.09 270) (effects (font (size 1.27 1.27)) (justify right bottom)))
@@
   (label "U1_PIN1?" (at 185.42 72.39 180) (effects (font (size 1.27 1.27)) (justify right bottom)))
   (wire (pts (xy 190.5 74.93) (xy 185.42 74.93)) (stroke (width 0) (type default) (color 0 0 0 0)))
-  (label "U1_PIN2?" (at 185.42 74.93 180) (effects (font (size 1.27 1.27)) (justify right bottom)))
+  (label "BAT+" (at 185.42 74.93 180) (effects (font (size 1.27 1.27)) (justify right bottom)))
+  (wire (pts (xy 205.74 72.39) (xy 210.82 72.39)) (stroke (width 0) (type default) (color 0 0 0 0)))
+  (label "GND" (at 210.82 72.39 0) (effects (font (size 1.27 1.27)) (justify left bottom)))
   (symbol (lib_id "Device:Battery_Cell") (at 243.84 76.2 0) (unit 1)
     (in_bom yes) (on_board yes)
@@
   )
   (symbol_instances
-    (path "/9b05b7dc-7754-4001-8e15-fcdc1db41cd4" (reference "USB1") (unit 1) (value "USB-C 6P") (footprint ""))
-    (path "/c8ade35c-b643-4500-a6ab-34073640b7ca" (reference "R8") (unit 1) (value "5.1k") (footprint ""))
-    (path "/7fad6f86-0fd0-406b-8c07-71ae9a50b1d4" (reference "R9") (unit 1) (value "5.1k") (footprint ""))
-    (path "/daee0bdf-3d93-422b-9745-2df6112686b6" (reference "R7") (unit 1) (value "1k") (footprint ""))
-    (path "/3528749a-0d55-4e88-9a33-6c3f8f472252" (reference "R6") (unit 1) (value "0") (footprint ""))
-    (path "/d4d82dd7-a8bc-4f68-b18b-7c93c167785f" (reference "C1") (unit 1) (value "?") (footprint ""))
-    (path "/54a6642d-6917-40c6-8811-0ae1bfe2c080" (reference "C2") (unit 1) (value "?") (footprint ""))
-    (path "/52bf3089-43d2-4f08-9e03-d9cad15fc638" (reference "U1") (unit 1) (value "unmarked") (footprint ""))
-    (path "/f36afff8-4c5f-4072-b8cc-51c613fee4cc" (reference "BT1") (unit 1) (value "Cell 3.7V") (footprint ""))
-    (path "/a75489c8-02f5-4a3a-993a-8081094067bb" (reference "M1") (unit 1) (value "Motor") (footprint ""))
-    (path "/1ecd8c17-4d74-4fda-b938-beb2e0bf8491" (reference "D2") (unit 1) (value "D (polarity unverified)") (footprint ""))
-    (path "/eb8dc780-c55e-4c22-b544-52863d6c9b6c" (reference "C3") (unit 1) (value "? 50V") (footprint ""))
-    (path "/654f2be0-54a4-403e-bcd5-3317a1f32dde" (reference "R2") (unit 1) (value "10k? (103)") (footprint ""))
-    (path "/c16795c8-90d2-47b3-bbf5-b7bc31cc2bae" (reference "C4") (unit 1) (value "?") (footprint ""))
-    (path "/98854181-dc7c-4fcc-8343-896481265c3e" (reference "R4") (unit 1) (value "0") (footprint ""))
-    (path "/3d56e0a2-a186-4ad0-8a04-49f1224ca1b3" (reference "K1") (unit 1) (value "Power button") (footprint ""))
-    (path "/90f0b3b7-00e1-43dd-a337-e1fe1252b0f4" (reference "LED4") (unit 1) (value "LED") (footprint ""))
-    (path "/be409e48-5134-4f5b-875e-dc909a5e3877" (reference "LED1") (unit 1) (value "LED") (footprint ""))
-    (path "/2f03de07-105c-41ef-8064-1228e8a71cf8" (reference "LED2") (unit 1) (value "LED") (footprint ""))
-    (path "/17de7004-1ec3-4055-9855-cc4829ea2370" (reference "LED3") (unit 1) (value "LED") (footprint ""))
-    (path "/f4c615f9-3582-4289-bdf8-1572f87d7c79" (reference "R1") (unit 1) (value "?") (footprint ""))
-    (path "/ccef422f-706c-4d7b-ae71-3912b54af635" (reference "R3") (unit 1) (value "0") (footprint ""))
-    (path "/7c201197-3cf0-49c9-81df-e68b69c1f682" (reference "R5") (unit 1) (value "0") (footprint ""))
+    (path "/fd8434d0-797c-4478-979c-593cf2b83bb4" (reference "USB1") (unit 1) (value "USB-C 6P") (footprint ""))
+    (path "/a65682fc-5228-4727-8d59-32f42a659b10" (reference "R8") (unit 1) (value "5.1k") (footprint ""))
+    (path "/2bb2cb31-e175-49d4-bba5-f6ab7a117297" (reference "R9") (unit 1) (value "5.1k") (footprint ""))
+    (path "/e0414cc6-1e7c-4227-b375-9c09e97f652c" (reference "R7") (unit 1) (value "1k") (footprint ""))
+    (path "/84fa530e-cf40-4058-818c-91e7545caae6" (reference "R6") (unit 1) (value "0") (footprint ""))
+    (path "/885e2d60-9bc9-4eb2-88c3-fb930a0043f4" (reference "C1") (unit 1) (value "?") (footprint ""))
+    (path "/541d5e67-b971-4340-9af3-5d0b5eb67501" (reference "C2") (unit 1) (value "?") (footprint ""))
+    (path "/90efda48-8a64-435a-b6d2-8670607dc818" (reference "U1") (unit 1) (value "unmarked") (footprint ""))
+    (path "/1ad6a8b9-58f7-4ae0-b031-c4a2b14b546a" (reference "BT1") (unit 1) (value "Cell 3.7V") (footprint ""))
+    (path "/8f85216f-4154-49c1-8aab-b48467181fdd" (reference "M1") (unit 1) (value "Motor") (footprint ""))
+    (path "/522fd18c-adb6-400a-b05b-e042f6a13dd6" (reference "D2") (unit 1) (value "D (polarity unverified)") (footprint ""))
+    (path "/a2a8cd08-2f2f-432e-a018-6ee175032896" (reference "C3") (unit 1) (value "? 50V") (footprint ""))
+    (path "/ef8e142c-1272-428d-9aec-0380c79d16ad" (reference "R2") (unit 1) (value "10k? (103)") (footprint ""))
+    (path "/d3149b96-40b6-4bc9-af76-e450c8a7f8fa" (reference "C4") (unit 1) (value "?") (footprint ""))
+    (path "/92e39e87-2a34-43d3-b745-c0c058f00e86" (reference "R4") (unit 1) (value "0") (footprint ""))
+    (path "/e2f0dbfa-c0a1-449e-8a8d-886e0f9850d1" (reference "K1") (unit 1) (value "Power button") (footprint ""))
+    (path "/61827d82-ea36-44a2-afd3-81e0e855848e" (reference "LED4") (unit 1) (value "LED") (footprint ""))
+    (path "/4845e1f3-d766-49f1-85ca-033ea14ae588" (reference "LED1") (unit 1) (value "LED") (footprint ""))
+    (path "/5ba94364-75d8-49b4-98f2-5e848842ed78" (reference "LED2") (unit 1) (value "LED") (footprint ""))
+    (path "/e790b24d-6ee5-451b-8bf7-f7ec608f93ab" (reference "LED3") (unit 1) (value "LED") (footprint ""))
+    (path "/c58e8aff-1a97-4d90-8baa-58c18cffe47b" (reference "R1") (unit 1) (value "?") (footprint ""))
+    (path "/58ff265a-aa5b-47e6-b060-fef9dd53caa4" (reference "R3") (unit 1) (value "0") (footprint ""))
+    (path "/966fe5d2-812b-4c14-acf3-f2db600e6cbd" (reference "R5") (unit 1) (value "0") (footprint ""))
   )
 )
